File: CNC-PCB-revamp.sch (KiCad schematic (older format))
At the start: 0 parts

Commit message: update,
Changed lines of the file:
@@
 $Descr A4 11693 8268
 encoding utf-8
-Sheet 1 4
+Sheet 1 5
 Title ""
 Date ""
@@
 F1 "STEP_MOTOR_DRIVER.sch" 50
 $EndSheet
+$Sheet
+S 9650 2100 1250 850
+U 5BFF1764
+F0 "POWER_SUPPLY" 50
+F1 "POWER_SUPPLY.sch" 50
+$EndSheet
 $EndSCHEMATC
