File: CNC-PCB-revamp.kicad_pcb (KiCad board)
At the start: 2 copper layers, 24 parts, among them J1 Conn_RPi_02_20, J10 Conn_02x12_Odd_Even, J2 Conn_02x03_Odd_Even, J3 Conn_02x03_Odd_Even, J4 Conn_02x03_Odd_Even, J5 Conn_01x04, J6 Conn_01x04, J7 Conn_01x04, J8 Conn_01x05, J9 Barrel_Jack_Switch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

Commit message: update,
Parts:
- added J11: Conn_01x02, Connector_JST:JST_XH_S02B-XH-A-1_1x02_P2.50mm_Horizontal, F.Cu at (120.4, 43.8)
- added J12: Conn_01x02, Connector_JST:JST_XH_S02B-XH-A-1_1x02_P2.50mm_Horizontal, F.Cu at (139.3, 42.9)
- added J13: Conn_01x02, Connector_JST:JST_XH_S02B-XH-A-1_1x02_P2.50mm_Horizontal, F.Cu at (157.9, 42.8)
- added J14: Conn_01x02, Connector_JST:JST_XH_S02B-XH-A-1_1x02_P2.50mm_Horizontal, F.Cu at (92.3, 43.7)
- added J15: Conn_01x02, Connector_JST:JST_XH_S02B-XH-A-1_1x02_P2.50mm_Horizontal, F.Cu at (102.1, 44.5)
- added J16: Conn_01x02, Connector_JST:JST_XH_S02B-XH-A-1_1x02_P2.50mm_Horizontal, F.Cu at (109.8, 44.8)
- added J17: Conn_01x02, Connector_JST:JST_XH_S02B-XH-A-1_1x02_P2.50mm_Horizontal, F.Cu at (129.6, 43.3)
- added J18: Conn_01x02, Connector_JST:JST_XH_S02B-XH-A-1_1x02_P2.50mm_Horizontal, F.Cu at (148.0, 42.8)
- added J19: Conn_01x02, Connector_JST:JST_XH_S02B-XH-A-1_1x02_P2.50mm_Horizontal, F.Cu at (166.8, 42.8)
- J5, J6, J7: footprint Connector_PinHeader_2.54mm:PinHeader_1x04_P2.54mm_Vertical -> Connector_JST:JST_XH_S04B-XH-A-1_1x04_P2.50mm_Horizontal
- R1, R2: moved to B.Cu
- moved J10 312.2 mm to (-163.6, 89.0), turned to 90 degrees
- moved H2 151.6 mm to (24.1, 133.8)
- moved H4 127.0 mm to (24.6, 29.7)
- moved J5 115.2 mm to (65.9, 110.7), turned to 90 degrees
- moved C1 108.0 mm to (45.7, 113.3), turned to 180 degrees
- moved H1 98.4 mm to (205.3, 136.1)
- moved U2 94.0 mm to (39.4, 97.9)
- moved J2 86.2 mm to (47.0, 106.9), turned to 180 degrees
- moved U1 52.6 mm to (96.5, 73.4), turned to 90 degrees
- moved J9 42.5 mm to (201.6, 50.0), turned to 180 degrees
- moved J7 42.1 mm to (193.0, 127.8), turned to 90 degrees
- moved J4 34.0 mm to (176.2, 123.0), turned to 180 degrees
- moved D1 33.2 mm to (29.0, 53.4), turned to 90 degrees
- moved R1 32.8 mm to (36.1, 51.9), turned to 180 degrees
- moved J3 32.3 mm to (156.1, 80.8), turned to 180 degrees
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Routing:
- net GND: track 0.00 -> 13.2 mm
- net Net-(J1-Pad10): track 0.00 -> 12.1 mm
- net Net-(D1-Pad2): track 0.00 -> 9.66 mm
