File: CNC-PCB-revamp.kicad_pcb (KiCad board)
At the start: 2 copper layers, 215 x 135 mm, 32 parts, among them J1 Conn_RPi_02_20, J11 X_LIMIT1, J12 Y_LIMIT1, J13 Z_LIMIT1, J14 PROBE, J15 START, J16 HOLD, J17 X_LIMIT2, J18 Y_LIMIT2, J19 Z_LIMIT2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

Commit message: update,
Parts:
- J1: moved to F.Cu
- moved J1 28.7 mm to (32.8, 20.1), turned to 90 degrees

Commit message: update,
Parts:
- moved H1 66.4 mm to (200.0, 70.0)
- moved H2 63.8 mm to (25.0, 70.0)
- moved H3 27.3 mm to (200.0, 30.0)
- moved J9 11.4 mm to (181.5, 62.5)
- moved H4 0.47 mm to (25.0, 30.0)
Changed lines of the file:
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@@
-(kicad_pcb (version 20171130) (host pcbnew 5.0.1-33cea8e~68~ubuntu18.04.1)
+(kicad_pcb (version 20171130) (host pcbnew 5.0.2-bee76a0~70~ubuntu18.04.1)
   (general
     (thickness 1.6)
@@
     (mod_text_size 1 1)
     (mod_text_width 0.15)
-    (pad_size 1.524 1.524)
-    (pad_drill 0.762)
+    (pad_size 5.4 5.4)
+    (pad_drill 2.7)
     (pad_to_mask_clearance 0.051)
     (solder_mask_min_width 0.25)
@@
   )
   (module Connector_BarrelJack:BarrelJack_Horizontal (layer F.Cu)
-    (at 190.37 69.61 180)
+    (at 181.5 62.5 180)
     (descr "DC Barrel Jack")
     (tags "Power Jack")
@@
   )
   (module MountingHole:MountingHole_2.7mm_M2.5_Pad (layer F.Cu)
-    (at 24.61 29.73)
+    (at 25 30)
     (descr "Mounting Hole 2.7mm, M2.5")
     (tags "mounting hole 2.7mm m2.5")
@@
   )
   (module MountingHole:MountingHole_2.7mm_M2.5_Pad (layer F.Cu)
-    (at 173.25 24.66)
+    (at 200 30)
     (descr "Mounting Hole 2.7mm, M2.5")
     (tags "mounting hole 2.7mm m2.5")
@@
   )
   (module MountingHole:MountingHole_2.7mm_M2.5_Pad (layer F.Cu)
-    (at 24.08 133.77)
+    (at 25 70)
     (descr "Mounting Hole 2.7mm, M2.5")
     (tags "mounting hole 2.7mm m2.5")
@@
   )
   (module MountingHole:MountingHole_2.7mm_M2.5_Pad (layer F.Cu)
-    (at 205.34 136.14)
+    (at 200 70)
     (descr "Mounting Hole 2.7mm, M2.5")
     (tags "mounting hole 2.7mm m2.5")

Commit message: update,
Parts:
- added C4: CP220uf,50V, Capacitor_SMD:CP_Elec_10x10.5, F.Cu at (-100.2, 40.2)
- added C5: C105,0805, Capacitor_SMD:C_0805_2012Metric_Pad1.15x1.40mm_HandSolder, F.Cu at (-76.4, 64.0)
- added C6: C105,0805, Capacitor_SMD:C_0805_2012Metric_Pad1.15x1.40mm_HandSolder, F.Cu at (-68.9, 64.0)
- added C7: C105,0805, Capacitor_SMD:C_0805_2012Metric_Pad1.15x1.40mm_HandSolder, F.Cu at (-72.7, 64.0)
- added C8: CP330uf,25V, Capacitor_SMD:CP_Elec_8x10.5, F.Cu at (-65.4, 40.3)
- added D2: SD_SS510, Diode_SMD:D_1206_3216Metric_Pad1.42x1.75mm_HandSolder, F.Cu at (-32.2, 10.1)
- added D3: SD_SS510, Diode_SMD:D_1206_3216Metric_Pad1.42x1.75mm_HandSolder, F.Cu at (-63.4, 55.2)
- added D4: SD_1N5817_SS12, Diode_SMD:D_1206_3216Metric_Pad1.42x1.75mm_HandSolder, F.Cu at (-58.4, 55.2)
- added J20: PWM_TO_MOTOR, Connector_PinHeader_2.54mm:PinHeader_1x02_P2.54mm_Vertical, F.Cu at (-33.5, 6.30)
- added L1: L_47UH,5A,1040, Inductor_SMD:L_Wuerth_HCI-1040, F.Cu at (-75.4, 70.7)
- added Q1: IRF540N, Package_TO_SOT_SMD:TO-263-2, F.Cu at (-27.0, 19.0)
- added R3: R330,0805, Resistor_SMD:R_0805_2012Metric_Pad1.15x1.40mm_HandSolder, F.Cu at (-23.8, 27.6)
- added R4: R102,0805, Resistor_SMD:R_0805_2012Metric_Pad1.15x1.40mm_HandSolder, F.Cu at (-26.7, 7.00)
- added R5: R103,0805, Resistor_SMD:R_0805_2012Metric_Pad1.15x1.40mm_HandSolder, F.Cu at (-16.9, 17.2)
- added R6: R103,0805, Resistor_SMD:R_0805_2012Metric_Pad1.15x1.40mm_HandSolder, F.Cu at (-60.3, 57.4)
- added R7: R333,0805, Resistor_SMD:R_0805_2012Metric_Pad1.15x1.40mm_HandSolder, F.Cu at (-64.1, 59.3)
- added R8: R332,0805, Resistor_SMD:R_0805_2012Metric_Pad1.15x1.40mm_HandSolder, F.Cu at (-64.1, 57.4)
- added U5: 4N35, Package_DIP:DIP-6_W7.62mm, F.Cu at (-28.5, 26.8)
- added U6: XL4015, Package_TO_SOT_SMD:TO-263-5_TabPin3, F.Cu at (-82.0, 40.4)
- J1: footprint Connector_PinSocket_2.54mm:PinSocket_2x20_P2.54mm_Vertical -> footprint-lib:Conn_RPi_02_20
- R1, R2: moved to F.Cu
- U1: footprint Module:Arduino_Nano -> footprint-lib:Arduino_Nano
- moved J9 166.5 mm to (30.9, 133.6), turned to 0 degrees
- moved J19 150.5 mm to (48.3, 126.5), turned to 0 degrees
- moved J13 136.2 mm to (57.1, 126.5), turned to 0 degrees
- moved J18 117.8 mm to (69.4, 126.5), turned to 0 degrees
- moved J12 106.3 mm to (78.1, 126.5), turned to 0 degrees
- moved J17 91.8 mm to (92.1, 126.5), turned to 0 degrees
- moved R2 86.6 mm to (-49.2, 57.2)
- moved J11 86.2 mm to (100.7, 126.5), turned to 0 degrees
- moved R1 82.2 mm to (-45.9, 57.2), turned to 0 degrees
- moved D1 77.4 mm to (-48.4, 55.2), turned to 0 degrees
- moved U1 73.5 mm to (38.3, 118.2), turned to 180 degrees
- moved J14 62.7 mm to (155.0, 41.5), turned to 90 degrees
- moved J1 58.8 mm to (85.8, 45.6), turned to 270 degrees
- moved J8 54.5 mm to (142.7, 24.4)
- moved J15 53.5 mm to (155.0, 51.3), turned to 90 degrees
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Connections:
- J9 pad 1: +VMot -> +24V
Routing:
- net Grbl_Tx: track 63.4 -> 0.00 mm
- net Net-(R4-Pad2): track 0.00 -> 45.5 mm
- net Probe: track 25.1 -> 0.00 mm
- net Start: track 23.5 -> 0.00 mm
- net Hold: track 19.2 -> 0.25 mm
- net +12V: track 0.00 -> 14.4 mm
- net Net-(D2-Pad2): track 0.00 -> 12.9 mm
- net Net-(J1-Pad10): track 12.1 -> 0.00 mm
- net Net-(D1-Pad2): track 9.66 -> 0.00 mm
- net Net-(D3-Pad1): track 0.00 -> 9.15 mm
- net Net-(J6-Pad1): track 8.89 -> 0.00 mm
- net Net-(J6-Pad3): track 8.89 -> 0.00 mm
- net Net-(J6-Pad4): track 8.89 -> 0.00 mm
- net Net-(J7-Pad2): track 7.91 -> 0.00 mm
- net Net-(J7-Pad3): track 7.90 -> 0.00 mm
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Other:
- board size 215 x 135 mm -> 150 x 135 mm

Commit message: update,
Parts:
- removed C1, C2, C3: CP47uf,35V, w_smd_cap:c_elec_5x5.3
- removed C4: CP220uf,50V, Capacitor_SMD:CP_Elec_10x10.5
- removed C5, C6, C7: C105,0805, Capacitor_SMD:C_0805_2012Metric_Pad1.15x1.40mm_HandSolder
- removed C8: CP330uf,25V, Capacitor_SMD:CP_Elec_8x10.5
- removed D1: SD_1N5819_SS14, Diode_SMD:D_1206_3216Metric_Pad1.42x1.75mm_HandSolder
- removed D2, D3: SD_SS510, Diode_SMD:D_1206_3216Metric_Pad1.42x1.75mm_HandSolder
- removed D4: SD_1N5817_SS12, Diode_SMD:D_1206_3216Metric_Pad1.42x1.75mm_HandSolder
- removed J11: X_LIMIT1, Connector_JST:JST_XH_S02B-XH-A-1_1x02_P2.50mm_Horizontal
- removed J12: Y_LIMIT1, Connector_JST:JST_XH_S02B-XH-A-1_1x02_P2.50mm_Horizontal
- removed J13: Z_LIMIT1, Connector_JST:JST_XH_S02B-XH-A-1_1x02_P2.50mm_Horizontal
- removed J17: X_LIMIT2, Connector_JST:JST_XH_S02B-XH-A-1_1x02_P2.50mm_Horizontal
- removed J18: Y_LIMIT2, Connector_JST:JST_XH_S02B-XH-A-1_1x02_P2.50mm_Horizontal
- removed J19: Z_LIMIT2, Connector_JST:JST_XH_S02B-XH-A-1_1x02_P2.50mm_Horizontal
- removed J2, J3, J4: Conn_02x03_Odd_Even, Connector_PinHeader_2.54mm:PinHeader_2x03_P2.54mm_Vertical
- removed J20: PWM_TO_MOTOR, Connector_PinHeader_2.54mm:PinHeader_1x02_P2.54mm_Vertical
- removed J5, J6, J7: Conn_01x04, Connector_JST:JST_XH_S04B-XH-A-1_1x04_P2.50mm_Horizontal
- removed L1: L_47UH,5A,1040, Inductor_SMD:L_Wuerth_HCI-1040
- removed Q1: IRF540N, Package_TO_SOT_SMD:TO-263-2
- removed R1: R102,0603, Resistor_SMD:R_0603_1608Metric_Pad1.05x0.95mm_HandSolder
- removed R2: R202,0603, Resistor_SMD:R_0603_1608Metric_Pad1.05x0.95mm_HandSolder
- removed R3: R330,0805, Resistor_SMD:R_0805_2012Metric_Pad1.15x1.40mm_HandSolder
- removed R4: R102,0805, Resistor_SMD:R_0805_2012Metric_Pad1.15x1.40mm_HandSolder
- removed R5, R6: R103,0805, Resistor_SMD:R_0805_2012Metric_Pad1.15x1.40mm_HandSolder
- removed R7: R333,0805, Resistor_SMD:R_0805_2012Metric_Pad1.15x1.40mm_HandSolder
- removed R8: R332,0805, Resistor_SMD:R_0805_2012Metric_Pad1.15x1.40mm_HandSolder
- removed U2, U3, U4: A4988_MODULE, Module:Pololu_Breakout-16_15.2x20.3mm
- removed U5: 4N35, Package_DIP:DIP-6_W7.62mm
- removed U6: XL4015, Package_TO_SOT_SMD:TO-263-5_TabPin3
- moved U1 94.8 mm to (119.4, 69.1)
- moved J9 69.7 mm to (29.0, 64.0)
- moved J14 37.3 mm to (127.1, 66.3), turned to 0 degrees
- moved J1 25.4 mm to (61.0, 40.2), turned to 180 degrees
- moved H1 20.0 mm to (150.0, 50.0)
- moved H2 20.0 mm to (25.0, 50.0)
- moved J15 19.3 mm to (142.8, 66.3), turned to 0 degrees
- moved J16 7.33 mm to (158.7, 66.3), turned to 0 degrees
Routing:
- net Net-(R4-Pad2): track 45.5 -> 0.00 mm
- net GND: track 29.0 -> 0.00 mm
- net +12V: track 14.4 -> 0.00 mm
- net Net-(D2-Pad2): track 12.9 -> 0.00 mm
- net Z_Limit: track 9.39 -> 0.00 mm
- net Y_Limit: track 9.24 -> 0.00 mm
- net Net-(D3-Pad1): track 9.15 -> 0.00 mm
- net X_Limit: track 9.13 -> 0.00 mm
- net Net-(Q1-Pad1): track 6.60 -> 0.00 mm
- net Net-(J3-Pad6): track 5.39 -> 0.00 mm
- net Net-(J3-Pad4): track 5.39 -> 0.00 mm
- net Net-(J3-Pad2): track 5.39 -> 0.00 mm
- net Net-(J2-Pad6): track 5.32 -> 0.00 mm
- net Net-(J2-Pad2): track 5.32 -> 0.00 mm
- net Net-(J2-Pad4): track 5.32 -> 0.00 mm
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Other:
- board size 150 x 135 mm -> 150 x 80 mm

Commit message: update,
Parts:
- added C1: CP47uf,35V, w_smd_cap:c_elec_5x5.3, F.Cu at (185.5, -20.5)
- added C2: CP47uf,35V, w_smd_cap:c_elec_5x5.3, F.Cu at (186.0, 32.5)
- added C3: CP47uf,35V, w_smd_cap:c_elec_5x5.3, F.Cu at (185.0, 7.00)
- added C4: CP220uf,50V, Capacitor_SMD:CP_Elec_10x10.5, F.Cu at (-64.7, 74.4)
- added C5: C105,0805, Capacitor_SMD:C_0805_2012Metric_Pad1.15x1.40mm_HandSolder, F.Cu at (-49.3, 67.5)
- added C6: C105,0805, Capacitor_SMD:C_0805_2012Metric_Pad1.15x1.40mm_HandSolder, F.Cu at (-45.6, 67.5)
- added C7: C105,0805, Capacitor_SMD:C_0805_2012Metric_Pad1.15x1.40mm_HandSolder, F.Cu at (-40.7, 60.9)
- added C8: CP330uf,25V, Capacitor_SMD:CP_Elec_8x10.5, F.Cu at (-48.8, 62.0)
- added D1: SD_1N5819_SS14, Diode_SMD:D_1206_3216Metric_Pad1.42x1.75mm_HandSolder, F.Cu at (-69.1, 84.8)
- added D2: SD_SS510, Diode_SMD:D_1206_3216Metric_Pad1.42x1.75mm_HandSolder, F.Cu at (-83.2, 107.8)
- added D3: SD_SS510, Diode_SMD:D_1206_3216Metric_Pad1.42x1.75mm_HandSolder, F.Cu at (-35.1, 58.7)
- added D4: SD_1N5817_SS12, Diode_SMD:D_1206_3216Metric_Pad1.42x1.75mm_HandSolder, F.Cu at (-40.1, 58.7)
- added J10: Mist, Connector_JST:JST_XH_S02B-XH-A-1_1x02_P2.50mm_Horizontal, F.Cu at (-108.2, 112.3)
- added J11: X_LIMIT1, Connector_JST:JST_XH_S02B-XH-A-1_1x02_P2.50mm_Horizontal, F.Cu at (-99.7, 99.7)
- added J12: Y_LIMIT1, Connector_JST:JST_XH_S02B-XH-A-1_1x02_P2.50mm_Horizontal, F.Cu at (-108.2, 99.7)
- added J13: Z_LIMIT1, Connector_JST:JST_XH_S02B-XH-A-1_1x02_P2.50mm_Horizontal, F.Cu at (-125.1, 112.3)
- added J17: X_LIMIT2, Connector_JST:JST_XH_S02B-XH-A-1_1x02_P2.50mm_Horizontal, F.Cu at (-99.7, 112.3)
- added J18: Y_LIMIT2, Connector_JST:JST_XH_S02B-XH-A-1_1x02_P2.50mm_Horizontal, F.Cu at (-116.6, 99.7)
- added J19: Z_LIMIT2, Connector_JST:JST_XH_S02B-XH-A-1_1x02_P2.50mm_Horizontal, F.Cu at (-133.5, 99.7)
- added J2: Conn_02x03_Odd_Even, Connector_PinHeader_2.54mm:PinHeader_2x03_P2.54mm_Vertical, F.Cu at (186.5, -27.5)
- added J20: PWM_TO_MOTOR, Connector_PinHeader_2.54mm:PinHeader_1x02_P2.54mm_Vertical, F.Cu at (-67.2, 105.3)
- added J21: Mist, Connector_JST:JST_XH_S02B-XH-A-1_1x02_P2.50mm_Horizontal, F.Cu at (-125.1, 99.7)
- added J22: Mist, Connector_JST:JST_XH_S02B-XH-A-1_1x02_P2.50mm_Horizontal, F.Cu at (-116.6, 112.3)
- added J23: Mist, Connector_JST:JST_XH_S02B-XH-A-1_1x02_P2.50mm_Horizontal, F.Cu at (-133.5, 112.3)
- added J3: Conn_02x03_Odd_Even, Connector_PinHeader_2.54mm:PinHeader_2x03_P2.54mm_Vertical, F.Cu at (187.5, 24.5)
- added J4: Conn_02x03_Odd_Even, Connector_PinHeader_2.54mm:PinHeader_2x03_P2.54mm_Vertical, F.Cu at (186.5, 0.50)
- added J5: Conn_01x04, Connector_JST:JST_XH_S04B-XH-A-1_1x04_P2.50mm_Horizontal, F.Cu at (199.0, -22.0)
- added J6: Conn_01x04, Connector_JST:JST_XH_S04B-XH-A-1_1x04_P2.50mm_Horizontal, F.Cu at (199.0, 31.0)
- added J7: Conn_01x04, Connector_JST:JST_XH_S04B-XH-A-1_1x04_P2.50mm_Horizontal, F.Cu at (199.5, 5.00)
- added L1: L_47UH,5A,1040, Inductor_SMD:L_Wuerth_HCI-1040, F.Cu at (-52.0, 74.2)
- added Q1: IRF540N, Package_TO_SOT_SMD:TO-263-2, F.Cu at (-77.4, 101.0)
- added R1: R102,0603, Resistor_SMD:R_0603_1608Metric_Pad1.05x0.95mm_HandSolder, F.Cu at (-66.6, 86.8)
- added R2: R202,0603, Resistor_SMD:R_0603_1608Metric_Pad1.05x0.95mm_HandSolder, F.Cu at (-70.0, 86.8)
- added R3: R330,0805, Resistor_SMD:R_0805_2012Metric_Pad1.15x1.40mm_HandSolder, F.Cu at (-71.4, 107.6)
- added R4: R102,0805, Resistor_SMD:R_0805_2012Metric_Pad1.15x1.40mm_HandSolder, F.Cu at (-75.1, 107.6)
- added R5: R103,0805, Resistor_SMD:R_0805_2012Metric_Pad1.15x1.40mm_HandSolder, F.Cu at (-78.9, 107.6)
- added R6: R103,0805, Resistor_SMD:R_0805_2012Metric_Pad1.15x1.40mm_HandSolder, F.Cu at (-37.0, 60.9)
- added R7: R333,0805, Resistor_SMD:R_0805_2012Metric_Pad1.15x1.40mm_HandSolder, F.Cu at (-40.7, 62.8)
- added R8: R332,0805, Resistor_SMD:R_0805_2012Metric_Pad1.15x1.40mm_HandSolder, F.Cu at (-53.1, 67.5)
- added U2: A4988_MODULE, Module:Pololu_Breakout-16_15.2x20.3mm, F.Cu at (178.8, -34.5)
- added U3: A4988_MODULE, Module:Pololu_Breakout-16_15.2x20.3mm, F.Cu at (179.6, 18.5)
- added U4: A4988_MODULE, Module:Pololu_Breakout-16_15.2x20.3mm, F.Cu at (178.6, -7.45)
- added U5: 4N35, Package_DIP:DIP-6_W7.62mm, F.Cu at (-67.9, 96.9)
- added U6: XL4015, Package_TO_SOT_SMD:TO-263-5_TabPin3, F.Cu at (-63.3, 63.2)
- moved J8 42.8 mm to (105.7, 2.89)
- moved U1 4.41 mm to (115.0, 68.5)
Routing:
- net +5V: track 0.00 -> 32.0 mm
- net GND: track 0.00 -> 23.5 mm
- net +VMot: track 0.00 -> 15.9 mm
- net Net-(J5-Pad3): track 0.00 -> 9.19 mm
- net Net-(J5-Pad1): track 0.00 -> 7.56 mm
- net Net-(J5-Pad2): track 0.00 -> 7.54 mm
- net Net-(J5-Pad4): track 0.00 -> 7.51 mm
- net Net-(J4-Pad6): track 0.00 -> 5.54 mm
- net Net-(J4-Pad4): track 0.00 -> 5.54 mm
- net Net-(J4-Pad2): track 0.00 -> 5.54 mm
- net Net-(J2-Pad4): track 0.00 -> 5.39 mm
- net Net-(J2-Pad2): track 0.00 -> 5.39 mm
- net Net-(J2-Pad6): track 0.00 -> 5.39 mm

Commit message: update,
Parts:
- moved J9 47.3 mm to (-11.5, 39.5)
- moved Q1 6.49 mm to (-78.0, 94.5), turned to 90 degrees
Changed lines of the file:
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@@
   )
   (module Package_TO_SOT_SMD:TO-263-2 (layer F.Cu)
-    (at -77.394999 100.965001)
+    (at -78 94.5 90)
     (descr "TO-263 / D2PAK / DDPAK SMD package, http://www.infineon.com/cms/en/product/packages/PG-TO263/PG-TO263-3-1/")
     (tags "D2PAK DDPAK TO-263 D2PAK-3 TO-263-3 SOT-404")
     (attr smd)
-    (fp_text reference Q1 (at 0 -6.65) (layer F.SilkS)
-      (effects (font (size 1 1) (thickness 0.15)))
-    )
-    (fp_text value IRF540N (at 0 6.65) (layer F.Fab)
+    (fp_text reference Q1 (at 0 -6.65 90) (layer F.SilkS)
+      (effects (font (size 1 1) (thickness 0.15)))
+    )
+    (fp_text value IRF540N (at 0 6.65 90) (layer F.Fab)
       (effects (font (size 1 1) (thickness 0.15)))
     )
@@
     (fp_line (start 8.32 5.65) (end 8.32 -5.65) (layer F.CrtYd) (width 0.05))
     (fp_line (start 8.32 -5.65) (end -8.32 -5.65) (layer F.CrtYd) (width 0.05))
-    (fp_text user %R (at 0 0) (layer F.Fab)
-      (effects (font (size 1 1) (thickness 0.15)))
-    )
-    (pad 1 smd rect (at -5.775 -2.54) (size 4.6 1.1) (layers F.Cu F.Paste F.Mask)
+    (fp_text user %R (at 0 0 90) (layer F.Fab)
+      (effects (font (size 1 1) (thickness 0.15)))
+    )
+    (pad 1 smd rect (at -5.775 -2.54 90) (size 4.6 1.1) (layers F.Cu F.Paste F.Mask)
       (net 74 "Net-(Q1-Pad1)"))
-    (pad 3 smd rect (at -5.775 2.54) (size 4.6 1.1) (layers F.Cu F.Paste F.Mask)
-      (net 1 GND))
-    (pad 2 smd rect (at 3.375 0) (size 9.4 10.8) (layers F.Cu F.Mask)
+    (pad 3 smd rect (at -5.775 2.54 90) (size 4.6 1.1) (layers F.Cu F.Paste F.Mask)
+      (net 1 GND))
+    (pad 2 smd rect (at 3.375 0 90) (size 9.4 10.8) (layers F.Cu F.Mask)
       (net 79 "Net-(D2-Pad2)"))
-    (pad "" smd rect (at 5.8 2.775) (size 4.55 5.25) (layers F.Paste))
-    (pad "" smd rect (at 0.95 -2.775) (size 4.55 5.25) (layers F.Paste))
-    (pad "" smd rect (at 5.8 -2.775) (size 4.55 5.25) (layers F.Paste))
-    (pad "" smd rect (at 0.95 2.775) (size 4.55 5.25) (layers F.Paste))
+    (pad "" smd rect (at 5.8 2.775 90) (size 4.55 5.25) (layers F.Paste))
+    (pad "" smd rect (at 0.95 -2.775 90) (size 4.55 5.25) (layers F.Paste))
+    (pad "" smd rect (at 5.8 -2.775 90) (size 4.55 5.25) (layers F.Paste))
+    (pad "" smd rect (at 0.95 2.775 90) (size 4.55 5.25) (layers F.Paste))
     (model ${KISYS3DMOD}/Package_TO_SOT_SMD.3dshapes/TO-263-2.wrl
       (at (xyz 0 0 0))
@@
   )
   (module Connector_BarrelJack:BarrelJack_Horizontal (layer F.Cu)
-    (at 29 64)
+    (at -11.5 39.5)
     (descr "DC Barrel Jack")
     (tags "Power Jack")
