File: STEP_MOTOR_DRIVER.sch (KiCad schematic (older format))
At the start: 12 parts, among them J2 Conn_02x03_Odd_Even, J3 Conn_02x03_Odd_Even, J4 Conn_02x03_Odd_Even, J5 Conn_01x04, J6 Conn_01x04, J7 Conn_01x04, U2 A4988_MODULE, U3 A4988_MODULE, U4 A4988_MODULE

Commit message: update,
Connections:
- net at J5.1 (Pin_1): now also U2.11 (1B); no longer U2.14 (2B)
- net at J5.2 (Pin_2): now also U2.12 (1A); no longer U2.13 (2A)
- net at J5.3 (Pin_3): now also U2.13 (2A); no longer U2.12 (1A)
- net at J5.4 (Pin_4): now also U2.14 (2B); no longer U2.11 (1B)
- net at J6.1 (Pin_1): now also U3.11 (1B); no longer U3.14 (2B)
- net at J6.2 (Pin_2): now also U3.12 (1A); no longer U3.13 (2A)
- net at J6.3 (Pin_3): now also U3.13 (2A); no longer U3.12 (1A)
- net at J6.4 (Pin_4): now also U3.14 (2B); no longer U3.11 (1B)
- net at J7.1 (Pin_1): now also U4.11 (1B); no longer U4.14 (2B)
- net at J7.2 (Pin_2): now also U4.12 (1A); no longer U4.13 (2A)
- net at J7.3 (Pin_3): now also U4.13 (2A); no longer U4.12 (1A)
- net at J7.4 (Pin_4): now also U4.14 (2B); no longer U4.11 (1B)
Changed lines of the file:
@@
 L Connector_Generic:Conn_01x04 J5
 U 1 1 5C0008F6
-P 7750 1650
-F 0 "J5" H 7830 1642 50  0000 L CNN
-F 1 "Conn_01x04" H 7830 1551 50  0000 L CNN
-F 2 "Connector_JST:JST_XH_S04B-XH-A-1_1x04_P2.50mm_Horizontal" H 7750 1650 50  0001 C CNN
-F 3 "~" H 7750 1650 50  0001 C CNN
-	1    7750 1650
-	1    0    0    -1
+P 7750 1750
+F 0 "J5" H 7830 1742 50  0000 L CNN
+F 1 "Conn_01x04" H 7830 1651 50  0000 L CNN
+F 2 "Connector_JST:JST_XH_S04B-XH-A-1_1x04_P2.50mm_Horizontal" H 7750 1750 50  0001 C CNN
+F 3 "~" H 7750 1750 50  0001 C CNN
+	1    7750 1750
+	1    0    0    1
 $EndComp
 Wire Wire Line
@@
 L Connector_Generic:Conn_01x04 J6
 U 1 1 5C002156
-P 7750 3600
-F 0 "J6" H 7830 3592 50  0000 L CNN
-F 1 "Conn_01x04" H 7830 3501 50  0000 L CNN
-F 2 "Connector_JST:JST_XH_S04B-XH-A-1_1x04_P2.50mm_Horizontal" H 7750 3600 50  0001 C CNN
-F 3 "~" H 7750 3600 50  0001 C CNN
-	1    7750 3600
-	1    0    0    -1
+P 7750 3700
+F 0 "J6" H 7830 3692 50  0000 L CNN
+F 1 "Conn_01x04" H 7830 3601 50  0000 L CNN
+F 2 "Connector_JST:JST_XH_S04B-XH-A-1_1x04_P2.50mm_Horizontal" H 7750 3700 50  0001 C CNN
+F 3 "~" H 7750 3700 50  0001 C CNN
+	1    7750 3700
+	1    0    0    1
 $EndComp
 Wire Wire Line
@@
 L Connector_Generic:Conn_01x04 J7
 U 1 1 5C004096
-P 7750 5450
-F 0 "J7" H 7830 5442 50  0000 L CNN
-F 1 "Conn_01x04" H 7830 5351 50  0000 L CNN
-F 2 "Connector_JST:JST_XH_S04B-XH-A-1_1x04_P2.50mm_Horizontal" H 7750 5450 50  0001 C CNN
-F 3 "~" H 7750 5450 50  0001 C CNN
-	1    7750 5450
-	1    0    0    -1
-$EndComp
-Wire Wire Line
+P 7750 5550
+F 0 "J7" H 7830 5542 50  0000 L CNN
+F 1 "Conn_01x04" H 7830 5451 50  0000 L CNN
+F 2 "Connector_JST:JST_XH_S04B-XH-A-1_1x04_P2.50mm_Horizontal" H 7750 5550 50  0001 C CNN
+F 3 "~" H 7750 5550 50  0001 C CNN
+	1    7750 5550
+	1    0    0    1
+$EndComp
+Wire Wire Line
