File: arduino_nano.sch (KiCad schematic (older format))
At the start: 1 part, among them U1 arduino_nano_v3

Commit message: update,
Parts:
- U1: footprint Module:Arduino_Nano -> footprint-lib:Arduino_Nano
Changed lines of the file:
@@
 F 0 "U1" H 5850 4515 50  0000 C CNN
 F 1 "arduino_nano_v3" H 5850 4424 50  0000 C CNN
-F 2 "Module:Arduino_Nano" H 5750 2400 50  0001 C CNN
+F 2 "footprint-lib:Arduino_Nano" H 5750 2400 50  0001 C CNN
 F 3 "" H 5850 3600 50  0001 C CNN
 	1    5850 3600
