File: rpi_conn.sch (KiCad schematic (older format))
At the start: 1 part

Commit message: update,
Parts:
- added D?: SD_1N5819_SS14, symbol taobao-sd:SD_1N5819_SS14
- added R?: R102,0603, symbol taobao-r:R102,0603
- added R?: R202,0603, symbol taobao-r:R202,0603
Connections:
- net at J?.10 (GPIO15): now also R?.1, R?.2
- net PWM0: now reaches J?.12 (GPIO18)
- net at J?.2 (5V): now also J?.4 (5V), D?.2 (A)
- net GND: now reaches J?.6 (Gound)
- net GND: now also J?.9 (Gound), R?.2
- net Grbl_Rx: now reaches J?.8 (GPIO14)
- new net +5V: D?.1 (K)
- new net Grbl_Tx: R?.1
Changed lines of the file:
@@
 	1    0    0    -1
 $EndComp
+$Comp
+L power:GND #PWR?
+U 1 1 5BFEFF23
+P 3950 3050
+F 0 "#PWR?" H 3950 2800 50  0001 C CNN
+F 1 "GND" H 3955 2877 50  0000 C CNN
+F 2 "" H 3950 3050 50  0001 C CNN
+F 3 "" H 3950 3050 50  0001 C CNN
+	1    3950 3050
+	1    0    0    -1
+$EndComp
+Wire Wire Line
+	4850 2750 3950 2750
+Wire Wire Line
+	3950 2750 3950 3050
+$Comp
+L taobao-sd:SD_1N5819_SS14 D?
+U 1 1 5BFF0494
+P 7850 2150
+F 0 "D?" V 7804 2218 50  0000 L CNN
+F 1 "SD_1N5819_SS14" V 7895 2218 50  0000 L CNN
+F 2 "" V 7850 2150 50  0001 C CNN
+F 3 "~" V 7850 2150 50  0001 C CNN
+	1    7850 2150
+	0    1    1    0
+$EndComp
+$Comp
+L tinkerforge:+5V #PWR?
+U 1 1 5BFF052E
+P 7850 1850
+F 0 "#PWR?" H 7850 1700 50  0001 C CNN
+F 1 "+5V" H 7865 2023 50  0000 C CNN
+F 2 "" H 7850 1850 50  0000 C CNN
+F 3 "" H 7850 1850 50  0000 C CNN
+	1    7850 1850
+	1    0    0    -1
+$EndComp
+Wire Wire Line
+	7850 1850 7850 2050
+Wire Wire Line
+	7850 2350 7850 2250
+Wire Wire Line
+	7250 2350 7850 2350
+Wire Wire Line
+	7250 2450 7850 2450
+Wire Wire Line
+	7850 2450 7850 2350
+Connection ~ 7850 2350
+$Comp
+L power:GND #PWR?
+U 1 1 5BFF05EE
+P 7850 2950
+F 0 "#PWR?" H 7850 2700 50  0001 C CNN
+F 1 "GND" H 7855 2777 50  0000 C CNN
+F 2 "" H 7850 2950 50  0001 C CNN
+F 3 "" H 7850 2950 50  0001 C CNN
+	1    7850 2950
+	1    0    0    -1
+$EndComp
+Wire Wire Line
+	7250 2550 7850 2550
+Wire Wire Line
+	7850 2550 7850 2950
+Wire Wire Line
+	8200 2650 7250 2650
+Text GLabel 8200 2650 2    50   Input ~ 0
+Grbl_Rx
+Text GLabel 8200 2850 2    50   Input ~ 0
+PWM0
+Wire Wire Line
+	8200 2850 7250 2850
+Text GLabel 8850 2300 2    50   Input ~ 0
+Grbl_Tx
+$Comp
+L taobao-r:R102,0603 R?
+U 1 1 5BFF09E7
+P 8800 2550
+F 0 "R?" H 8859 2596 50  0000 L CNN
+F 1 "R102,0603" H 8859 2505 50  0000 L CNN
+F 2 "" H 8800 2550 50  0001 C CNN
+F 3 "~" H 8800 2550 50  0001 C CNN
+	1    8800 2550
+	1    0    0    -1
+$EndComp
+$Comp
+L taobao-r:R202,0603 R?
+U 1 1 5BFF0B07
+P 8800 2950
+F 0 "R?" H 8859 2996 50  0000 L CNN
+F 1 "R202,0603" H 8859 2905 50  0000 L CNN
+F 2 "" H 8800 2950 50  0001 C CNN
+F 3 "~" H 8800 2950 50  0001 C CNN
+	1    8800 2950
+	1    0    0    -1
+$EndComp
+$Comp
+L power:GND #PWR?
+U 1 1 5BFF0BB8
+P 8800 3300
+F 0 "#PWR?" H 8800 3050 50  0001 C CNN
+F 1 "GND" H 8805 3127 50  0000 C CNN
+F 2 "" H 8800 3300 50  0001 C CNN
+F 3 "" H 8800 3300 50  0001 C CNN
+	1    8800 3300
+	1    0    0    -1
+$EndComp
+Wire Wire Line
+	7250 2750 8800 2750
+Wire Wire Line
+	8800 2750 8800 2650
+Wire Wire Line
+	8800 2750 8800 2850
+Connection ~ 8800 2750
+Wire Wire Line
+	8800 2450 8800 2300
+Wire Wire Line
+	8800 2300 8850 2300
+Wire Wire Line
+	8800 3050 8800 3300
 $EndSCHEMATC

Commit message: update,
Parts:
- removed J?: Conn_RPi_02_20, symbol taobao-components:Conn_RPi_02_20
- removed R?: R102,0603, symbol taobao-r:R102,0603
- added J1: Conn_RPi_02_20, Connector_PinSocket_2.54mm:PinSocket_2x20_P2.54mm_Vertical, symbol taobao-components:Conn_RPi_02_20
- added R1: R102,0603, Resistor_SMD:R_0603_1608Metric_Pad1.05x0.95mm_HandSolder, symbol taobao-r:R102,0603
- D1: renamed from D?; footprint (none) -> Diode_SMD:D_1206_3216Metric_Pad1.42x1.75mm_HandSolder
- R2: renamed from R?; footprint (none) -> Resistor_SMD:R_0603_1608Metric_Pad1.05x0.95mm_HandSolder
Connections:
- net GND: now also J1.6 (Gound), J1.9 (Gound)
- net Grbl_Rx: now also J1.8 (GPIO14)
- net Grbl_Tx: now also R1.1
- net PWM0: now also J1.12 (GPIO18)
- net at R2.1: now also J1.10 (GPIO15), R1.2
- net at D1.2 (A): now also J1.2 (5V), J1.4 (5V)
Changed lines of the file:
@@
 $Descr A4 11693 8268
 encoding utf-8
-Sheet 2 4
+Sheet 2 5
 Title ""
 Date ""
@@
 $EndDescr
 $Comp
-L taobao-components:Conn_RPi_02_20 J?
-U 1 1 5BFEA9EE
-P 6100 3350
-AR Path="/5BFEA9D7/5BFEA9EE" Ref="J?"  Part="1"
-AR Path="/5BFEAB84/5BFEA9EE" Ref="J?"  Part="1"
-F 0 "J?" H 6050 4615 50  0000 C CNN
-F 1 "Conn_RPi_02_20" H 6050 4524 50  0000 C CNN
-F 2 "" H 6100 2400 50  0001 C CNN
-F 3 "" H 6100 2400 50  0001 C CNN
-	1    6100 3350
-	1    0    0    -1
-$EndComp
-$Comp
-L power:GND #PWR?
+L power:GND #PWR0101
 U 1 1 5BFEFF23
 P 3950 3050
-F 0 "#PWR?" H 3950 2800 50  0001 C CNN
+F 0 "#PWR0101" H 3950 2800 50  0001 C CNN
 F 1 "GND" H 3955 2877 50  0000 C CNN
 F 2 "" H 3950 3050 50  0001 C CNN
@@
 	3950 2750 3950 3050
 $Comp
-L taobao-sd:SD_1N5819_SS14 D?
+L taobao-sd:SD_1N5819_SS14 D1
 U 1 1 5BFF0494
 P 7850 2150
-F 0 "D?" V 7804 2218 50  0000 L CNN
+F 0 "D1" V 7804 2218 50  0000 L CNN
 F 1 "SD_1N5819_SS14" V 7895 2218 50  0000 L CNN
-F 2 "" V 7850 2150 50  0001 C CNN
+F 2 "Diode_SMD:D_1206_3216Metric_Pad1.42x1.75mm_HandSolder" V 7850 2150 50  0001 C CNN
 F 3 "~" V 7850 2150 50  0001 C CNN
 	1    7850 2150
@@
 $EndComp
 $Comp
-L tinkerforge:+5V #PWR?
+L tinkerforge:+5V #PWR0102
 U 1 1 5BFF052E
 P 7850 1850
-F 0 "#PWR?" H 7850 1700 50  0001 C CNN
+F 0 "#PWR0102" H 7850 1700 50  0001 C CNN
 F 1 "+5V" H 7865 2023 50  0000 C CNN
 F 2 "" H 7850 1850 50  0000 C CNN
@@
 Connection ~ 7850 2350
 $Comp
-L power:GND #PWR?
+L power:GND #PWR0103
 U 1 1 5BFF05EE
 P 7850 2950
-F 0 "#PWR?" H 7850 2700 50  0001 C CNN
+F 0 "#PWR0103" H 7850 2700 50  0001 C CNN
 F 1 "GND" H 7855 2777 50  0000 C CNN
 F 2 "" H 7850 2950 50  0001 C CNN
@@
 Grbl_Tx
 $Comp
-L taobao-r:R102,0603 R?
-U 1 1 5BFF09E7
-P 8800 2550
-F 0 "R?" H 8859 2596 50  0000 L CNN
-F 1 "R102,0603" H 8859 2505 50  0000 L CNN
-F 2 "" H 8800 2550 50  0001 C CNN
-F 3 "~" H 8800 2550 50  0001 C CNN
-	1    8800 2550
-	1    0    0    -1
-$EndComp
-$Comp
-L taobao-r:R202,0603 R?
+L taobao-r:R202,0603 R2
 U 1 1 5BFF0B07
 P 8800 2950
-F 0 "R?" H 8859 2996 50  0000 L CNN
+F 0 "R2" H 8859 2996 50  0000 L CNN
 F 1 "R202,0603" H 8859 2905 50  0000 L CNN
-F 2 "" H 8800 2950 50  0001 C CNN
+F 2 "Resistor_SMD:R_0603_1608Metric_Pad1.05x0.95mm_HandSolder" H 8800 2950 50  0001 C CNN
 F 3 "~" H 8800 2950 50  0001 C CNN
 	1    8800 2950
@@
 $EndComp
 $Comp
-L power:GND #PWR?
+L power:GND #PWR0104
 U 1 1 5BFF0BB8
 P 8800 3300
-F 0 "#PWR?" H 8800 3050 50  0001 C CNN
+F 0 "#PWR0104" H 8800 3050 50  0001 C CNN
 F 1 "GND" H 8805 3127 50  0000 C CNN
 F 2 "" H 8800 3300 50  0001 C CNN
@@
 Wire Wire Line
 	8800 3050 8800 3300
+$Comp
+L taobao-r:R102,0603 R1
+U 1 1 5C0117DA
+P 8800 2550
+F 0 "R1" H 8859 2596 50  0000 L CNN
+F 1 "R102,0603" H 8859 2505 50  0000 L CNN
+F 2 "Resistor_SMD:R_0603_1608Metric_Pad1.05x0.95mm_HandSolder" H 8800 2550 50  0001 C CNN
+F 3 "~" H 8800 2550 50  0001 C CNN
+	1    8800 2550
+	1    0    0    -1
+$EndComp
+$Comp
+L taobao-components:Conn_RPi_02_20 J1
+U 1 1 5C0226DB
+P 6100 3350
+F 0 "J1" H 6050 4615 50  0000 C CNN
+F 1 "Conn_RPi_02_20" H 6050 4524 50  0000 C CNN
+F 2 "Connector_PinSocket_2.54mm:PinSocket_2x20_P2.54mm_Vertical" H 6100 2400 50  0001 C CNN
+F 3 "" H 6100 2400 50  0001 C CNN
+	1    6100 3350
+	1    0    0    -1
+$EndComp
 $EndSCHEMATC
