File: rpi_conn.sch (KiCad schematic (older format))
At the start: 4 parts, among them J1 Conn_RPi_02_20

Commit message: update,
Parts:
- J1: footprint Connector_PinSocket_2.54mm:PinSocket_2x20_P2.54mm_Vertical -> footprint-lib:Conn_RPi_02_20
Changed lines of the file:
@@
 F 0 "J1" H 6050 4615 50  0000 C CNN
 F 1 "Conn_RPi_02_20" H 6050 4524 50  0000 C CNN
-F 2 "Connector_PinSocket_2.54mm:PinSocket_2x20_P2.54mm_Vertical" H 6100 2400 50  0001 C CNN
+F 2 "footprint-lib:Conn_RPi_02_20" H 6100 2400 50  0001 C CNN
 F 3 "" H 6100 2400 50  0001 C CNN
 	1    6100 3350
