File: POWER_SUPPLY.sch (KiCad schematic (older format))
At the start: 16 parts, among them J10 Conn_02x12_Odd_Even, J11 X_LIMIT1, J12 Y_LIMIT1, J13 Z_LIMIT1, J14 PROBE, J15 START, J16 HOLD, J17 X_LIMIT2, J18 Y_LIMIT2, J19 Z_LIMIT2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

Commit message: update,
Connections:
- net +VMot renamed +24V
Changed lines of the file:
@@
 	1    0    0    -1
 $EndComp
-$Comp
-L taobao-components:+VMot #PWR0122
-U 1 1 5BFF3CE7
-P 4200 1450
-F 0 "#PWR0122" H 4200 1300 50  0001 C CNN
-F 1 "+VMot" H 4215 1623 50  0000 C CNN
-F 2 "" H 4200 1450 50  0000 C CNN
-F 3 "" H 4200 1450 50  0000 C CNN
-	1    4200 1450
-	1    0    0    -1
-$EndComp
 Wire Wire Line
 	4200 1450 4200 1700
@@
 Wire Wire Line
 	3950 1900 4200 1900
+$Comp
+L power:+24V #PWR?
+U 1 1 5C008C1F
+P 4200 1450
+F 0 "#PWR?" H 4200 1300 50  0001 C CNN
+F 1 "+24V" H 4250 1650 50  0000 C CNN
+F 2 "" H 4200 1450 50  0001 C CNN
+F 3 "" H 4200 1450 50  0001 C CNN
+	1    4200 1450
+	1    0    0    -1
+$EndComp
 $EndSCHEMATC
