File: POWER_SUPPLY.sch (KiCad schematic (older format))
At the start: 16 parts, among them J10 Conn_02x12_Odd_Even, J11 X_LIMIT1, J12 Y_LIMIT1, J13 Z_LIMIT1, J14 PROBE, J15 START, J16 HOLD, J17 X_LIMIT2, J18 Y_LIMIT2, J19 Z_LIMIT2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

Commit message: update,
Parts:
- removed J9: Barrel_Jack_Switch, Connector_BarrelJack:BarrelJack_Horizontal, symbol Connector:Barrel_Jack_Switch
Changed lines of the file:
@@
 $EndDescr
 $Comp
-L Connector:Barrel_Jack_Switch J9
-U 1 1 5BFF19AA
-P 3650 1800
-AR Path="/5BFF1764/5BFF19AA" Ref="J9"  Part="1"
-AR Path="/5C064586/5BFF19AA" Ref="J?"  Part="1"
-F 0 "J?" H 3705 2117 50  0000 C CNN
-F 1 "Barrel_Jack_Switch" H 3705 2026 50  0000 C CNN
-F 2 "Connector_BarrelJack:BarrelJack_Horizontal" H 3700 1760 50  0001 C CNN
-F 3 "~" H 3700 1760 50  0001 C CNN
-	1    3650 1800
-	1    0    0    -1
-$EndComp
-Wire Wire Line
-	4200 1450 4200 1700
-Wire Wire Line
-	4200 1700 3950 1700
-$Comp
-L power:GND #PWR0123
-U 1 1 5BFF3D4E
-P 4200 2150
-AR Path="/5BFF1764/5BFF3D4E" Ref="#PWR0123"  Part="1"
-AR Path="/5C064586/5BFF3D4E" Ref="#PWR?"  Part="1"
-F 0 "#PWR?" H 4200 1900 50  0001 C CNN
-F 1 "GND" H 4205 1977 50  0000 C CNN
-F 2 "" H 4200 2150 50  0001 C CNN
-F 3 "" H 4200 2150 50  0001 C CNN
-	1    4200 2150
-	1    0    0    -1
-$EndComp
-Wire Wire Line
-	4200 1900 4200 2150
-$Comp
 L Mechanical:MountingHole_Pad H1
 U 1 1 5BFF4033
@@
 AR Path="/5BFF1764/5BFF4033" Ref="H1"  Part="1"
 AR Path="/5C064586/5BFF4033" Ref="H?"  Part="1"
-F 0 "H?" V 6750 4351 50  0000 L CNN
+F 0 "H1" V 6750 4351 50  0000 L CNN
 F 1 "MountingHole_Pad" V 6750 4260 50  0000 L CNN
 F 2 "MountingHole:MountingHole_2.7mm_M2.5_Pad" H 6650 4300 50  0001 C CNN
@@
 AR Path="/5BFF1764/5BFF40E1" Ref="H2"  Part="1"
 AR Path="/5C064586/5BFF40E1" Ref="H?"  Part="1"
-F 0 "H?" V 7050 4351 50  0000 L CNN
+F 0 "H2" V 7050 4351 50  0000 L CNN
 F 1 "MountingHole_Pad" V 7050 4260 50  0000 L CNN
 F 2 "MountingHole:MountingHole_2.7mm_M2.5_Pad" H 6950 4300 50  0001 C CNN
@@
 AR Path="/5BFF1764/5BFF40FF" Ref="H3"  Part="1"
 AR Path="/5C064586/5BFF40FF" Ref="H?"  Part="1"
-F 0 "H?" V 7350 4351 50  0000 L CNN
+F 0 "H3" V 7350 4351 50  0000 L CNN
 F 1 "MountingHole_Pad" V 7350 4260 50  0000 L CNN
 F 2 "MountingHole:MountingHole_2.7mm_M2.5_Pad" H 7250 4300 50  0001 C CNN
@@
 AR Path="/5BFF1764/5BFF4125" Ref="H4"  Part="1"
 AR Path="/5C064586/5BFF4125" Ref="H?"  Part="1"
-F 0 "H?" V 7600 4351 50  0000 L CNN
+F 0 "H4" V 7600 4351 50  0000 L CNN
 F 1 "MountingHole_Pad" V 7600 4260 50  0000 L CNN
 F 2 "MountingHole:MountingHole_2.7mm_M2.5_Pad" H 7500 4300 50  0001 C CNN
@@
 AR Path="/5BFF1764/5BFF421C" Ref="#PWR0124"  Part="1"
 AR Path="/5C064586/5BFF421C" Ref="#PWR?"  Part="1"
-F 0 "#PWR?" H 7100 4350 50  0001 C CNN
+F 0 "#PWR0124" H 7100 4350 50  0001 C CNN
 F 1 "GND" H 7105 4427 50  0000 C CNN
 F 2 "" H 7100 4600 50  0001 C CNN
@@
 AR Path="/5BFF1764/5BFF4535" Ref="J10"  Part="1"
 AR Path="/5C064586/5BFF4535" Ref="J?"  Part="1"
-F 0 "J?" H 7200 2617 50  0000 C CNN
+F 0 "J10" H 7200 2617 50  0000 C CNN
 F 1 "Conn_02x12_Odd_Even" H 7200 2526 50  0000 C CNN
 F 2 "Connector_PinHeader_2.54mm:PinHeader_2x12_P2.54mm_Vertical" H 7150 1900 50  0001 C CNN
@@
 AR Path="/5BFF1764/5BFF45EC" Ref="#PWR0125"  Part="1"
 AR Path="/5C064586/5BFF45EC" Ref="#PWR?"  Part="1"
-F 0 "#PWR?" H 6600 2550 50  0001 C CNN
+F 0 "#PWR0125" H 6600 2550 50  0001 C CNN
 F 1 "GND" H 6605 2627 50  0000 C CNN
 F 2 "" H 6600 2800 50  0001 C CNN
@@
 AR Path="/5BFF1764/5BFF6CCC" Ref="#PWR0126"  Part="1"
 AR Path="/5C064586/5BFF6CCC" Ref="#PWR?"  Part="1"
-F 0 "#PWR?" H 8600 1500 50  0001 C CNN
+F 0 "#PWR0126" H 8600 1500 50  0001 C CNN
 F 1 "+5V" H 8615 1823 50  0000 C CNN
 F 2 "" H 8600 1650 50  0000 C CNN
@@
 AR Path="/5BFF1764/5BFF8AAE" Ref="J8"  Part="1"
 AR Path="/5C064586/5BFF8AAE" Ref="J?"  Part="1"
-F 0 "J?" H 3020 4467 50  0000 C CNN
+F 0 "J8" H 3020 4467 50  0000 C CNN
 F 1 "MOTOR" H 3020 4376 50  0000 C CNN
 F 2 "Connector_JST:JST_XH_S05B-XH-A-1_1x05_P2.50mm_Horizontal" H 3100 4050 50  0001 C CNN
@@
 AR Path="/5BFF1764/5BFFB401" Ref="#PWR0127"  Part="1"
 AR Path="/5C064586/5BFFB401" Ref="#PWR?"  Part="1"
-F 0 "#PWR?" H 4250 4000 50  0001 C CNN
+F 0 "#PWR0127" H 4250 4000 50  0001 C CNN
 F 1 "+5V" H 4265 4323 50  0000 C CNN
 F 2 "" H 4250 4150 50  0000 C CNN
@@
 AR Path="/5BFF1764/5BFFBFD9" Ref="#PWR0128"  Part="1"
 AR Path="/5C064586/5BFFBFD9" Ref="#PWR?"  Part="1"
-F 0 "#PWR?" H 4150 3400 50  0001 C CNN
+F 0 "#PWR0128" H 4150 3400 50  0001 C CNN
 F 1 "GND" H 4155 3477 50  0000 C CNN
 F 2 "" H 4150 3650 50  0001 C CNN
@@
 AR Path="/5BFF1764/5C030BBA" Ref="J11"  Part="1"
 AR Path="/5C064586/5C030BBA" Ref="J?"  Part="1"
-F 0 "J?" H 9700 850 50  0000 C CNN
-F 1 "X_LIMIT1" H 9900 750 50  0000 C CNN
+F 0 "J11" H 9750 850 50  0000 C CNN
+F 1 "X_LIMIT1" H 9850 750 50  0000 C CNN
 F 2 "Connector_JST:JST_XH_S02B-XH-A-1_1x02_P2.50mm_Horizontal" H 9600 850 50  0001 C CNN
 F 3 "~" H 9600 850 50  0001 C CNN
@@
 AR Path="/5BFF1764/5C0318FB" Ref="J12"  Part="1"
 AR Path="/5C064586/5C0318FB" Ref="J?"  Part="1"
-F 0 "J?" H 9680 1192 50  0000 L CNN
+F 0 "J12" H 9680 1192 50  0000 L CNN
 F 1 "Y_LIMIT1" H 9680 1101 50  0000 L CNN
 F 2 "Connector_JST:JST_XH_S02B-XH-A-1_1x02_P2.50mm_Horizontal" H 9600 1200 50  0001 C CNN
@@
 AR Path="/5BFF1764/5C031931" Ref="J13"  Part="1"
 AR Path="/5C064586/5C031931" Ref="J?"  Part="1"
-F 0 "J?" H 9680 1492 50  0000 L CNN
+F 0 "J13" H 9680 1492 50  0000 L CNN
 F 1 "Z_LIMIT1" H 9680 1401 50  0000 L CNN
 F 2 "Connector_JST:JST_XH_S02B-XH-A-1_1x02_P2.50mm_Horizontal" H 9600 1500 50  0001 C CNN
@@
 AR Path="/5BFF1764/5C03426F" Ref="J14"  Part="1"
 AR Path="/5C064586/5C03426F" Ref="J?"  Part="1"
-F 0 "J?" H 9680 4192 50  0000 L CNN
+F 0 "J14" H 9680 4192 50  0000 L CNN
 F 1 "PROBE" H 9680 4101 50  0000 L CNN
 F 2 "Connector_JST:JST_XH_S02B-XH-A-1_1x02_P2.50mm_Horizontal" H 9600 4200 50  0001 C CNN
@@
 AR Path="/5BFF1764/5C0359F8" Ref="J15"  Part="1"
 AR Path="/5C064586/5C0359F8" Ref="J?"  Part="1"
-F 0 "J?" H 9680 4492 50  0000 L CNN
+F 0 "J15" H 9680 4492 50  0000 L CNN
 F 1 "START" H 9680 4401 50  0000 L CNN
 F 2 "Connector_JST:JST_XH_S02B-XH-A-1_1x02_P2.50mm_Horizontal" H 9600 4500 50  0001 C CNN
@@
 AR Path="/5BFF1764/5C03E431" Ref="J16"  Part="1"
 AR Path="/5C064586/5C03E431" Ref="J?"  Part="1"
-F 0 "J?" H 9680 4792 50  0000 L CNN
+F 0 "J16" H 9680 4792 50  0000 L CNN
 F 1 "HOLD" H 9680 4701 50  0000 L CNN
 F 2 "Connector_JST:JST_XH_S02B-XH-A-1_1x02_P2.50mm_Horizontal" H 9600 4800 50  0001 C CNN
@@
 AR Path="/5BFF1764/5C03F42E" Ref="#PWR0129"  Part="1"
 AR Path="/5C064586/5C03F42E" Ref="#PWR?"  Part="1"
-F 0 "#PWR?" H 9950 4900 50  0001 C CNN
+F 0 "#PWR0129" H 9950 4900 50  0001 C CNN
 F 1 "GND" H 9955 4977 50  0000 C CNN
 F 2 "" H 9950 5150 50  0001 C CNN
@@
 AR Path="/5BFF1764/5C0541C9" Ref="J17"  Part="1"
 AR Path="/5C064586/5C0541C9" Ref="J?"  Part="1"
-F 0 "J?" H 9650 2350 50  0000 C CNN
-F 1 "X_LIMIT2" H 9850 2250 50  0000 C CNN
+F 0 "J17" H 9700 2350 50  0000 C CNN
+F 1 "X_LIMIT2" H 9800 2250 50  0000 C CNN
 F 2 "Connector_JST:JST_XH_S02B-XH-A-1_1x02_P2.50mm_Horizontal" H 9550 2350 50  0001 C CNN
 F 3 "~" H 9550 2350 50  0001 C CNN
@@
 AR Path="/5BFF1764/5C0541D2" Ref="J18"  Part="1"
 AR Path="/5C064586/5C0541D2" Ref="J?"  Part="1"
-F 0 "J?" H 9630 2692 50  0000 L CNN
+F 0 "J18" H 9630 2692 50  0000 L CNN
 F 1 "Y_LIMIT2" H 9630 2601 50  0000 L CNN
 F 2 "Connector_JST:JST_XH_S02B-XH-A-1_1x02_P2.50mm_Horizontal" H 9550 2700 50  0001 C CNN
@@
 AR Path="/5BFF1764/5C0541D8" Ref="J19"  Part="1"
 AR Path="/5C064586/5C0541D8" Ref="J?"  Part="1"
-F 0 "J?" H 9630 2992 50  0000 L CNN
+F 0 "J19" H 9630 2992 50  0000 L CNN
 F 1 "Z_LIMIT2" H 9630 2901 50  0000 L CNN
 F 2 "Connector_JST:JST_XH_S02B-XH-A-1_1x02_P2.50mm_Horizontal" H 9550 3000 50  0001 C CNN
@@
 AR Path="/5BFF1764/5C055B77" Ref="#PWR0130"  Part="1"
 AR Path="/5C064586/5C055B77" Ref="#PWR?"  Part="1"
-F 0 "#PWR?" H 9950 1600 50  0001 C CNN
+F 0 "#PWR0130" H 9950 1600 50  0001 C CNN
 F 1 "GND" H 9955 1677 50  0000 C CNN
 F 2 "" H 9950 1850 50  0001 C CNN
@@
 AR Path="/5BFF1764/5C0573EE" Ref="#PWR0131"  Part="1"
 AR Path="/5C064586/5C0573EE" Ref="#PWR?"  Part="1"
-F 0 "#PWR?" H 9900 3100 50  0001 C CNN
+F 0 "#PWR0131" H 9900 3100 50  0001 C CNN
 F 1 "GND" H 9905 3177 50  0000 C CNN
 F 2 "" H 9900 3350 50  0001 C CNN
@@
 	9900 3100 9900 3350
 Connection ~ 9900 3100
-Wire Wire Line
-	3950 1900 4200 1900
-$Comp
-L power:+24V #PWR?
-U 1 1 5C008C1F
-P 4200 1450
-AR Path="/5BFF1764/5C008C1F" Ref="#PWR?"  Part="1"
-AR Path="/5C064586/5C008C1F" Ref="#PWR?"  Part="1"
-F 0 "#PWR?" H 4200 1300 50  0001 C CNN
-F 1 "+24V" H 4250 1650 50  0000 C CNN
-F 2 "" H 4200 1450 50  0001 C CNN
-F 3 "" H 4200 1450 50  0001 C CNN
-	1    4200 1450
-	1    0    0    -1
-$EndComp
 $EndSCHEMATC

Commit message: update,
Parts:
- removed J10: Conn_02x12_Odd_Even, Connector_PinHeader_2.54mm:PinHeader_2x12_P2.54mm_Vertical, symbol Connector_Generic:Conn_02x12_Odd_Even
- added J? (x4): Mist, Connector_JST:JST_XH_S02B-XH-A-1_1x02_P2.50mm_Horizontal, symbol Connector_Generic:Conn_01x02
Connections:
- net A6: now also J?.1 (Pin_1)
- net A7: now also J?.1 (Pin_1)
- net Flood: now also J?.1 (Pin_1)
- net GND: now also J?.2 (Pin_2), J?.2 (Pin_2), J?.2 (Pin_2), J?.2 (Pin_2)
- net Mist: now also J?.1 (Pin_1)
Other:
- moved on the sheet: H1, H2, H3, H4

Commit message: update,
Parts:
- gave numbers to parts that had none: 4
Changed lines of the file:
@@
 Connection ~ 9900 3100
 $Comp
-L Connector_Generic:Conn_01x02 J?
+L Connector_Generic:Conn_01x02 J21
 U 1 1 5C06FF5E
 P 7050 2750
-AR Path="/5BFF1764/5C06FF5E" Ref="J?"  Part="1"
+AR Path="/5BFF1764/5C06FF5E" Ref="J21"  Part="1"
 AR Path="/5C064586/5C06FF5E" Ref="J?"  Part="1"
-F 0 "J?" H 7130 2742 50  0000 L CNN
+F 0 "J21" H 7130 2742 50  0000 L CNN
 F 1 "Mist" H 7130 2651 50  0000 L CNN
 F 2 "Connector_JST:JST_XH_S02B-XH-A-1_1x02_P2.50mm_Horizontal" H 7050 2750 50  0001 C CNN
@@
 	7400 2850 7400 3150
 $Comp
-L power:GND #PWR?
+L power:GND #PWR0125
 U 1 1 5C0719A4
 P 7400 3150
-F 0 "#PWR?" H 7400 2900 50  0001 C CNN
+F 0 "#PWR0125" H 7400 2900 50  0001 C CNN
 F 1 "GND" H 7450 2950 50  0000 C CNN
 F 2 "" H 7400 3150 50  0001 C CNN
@@
 $EndComp
 $Comp
-L Connector_Generic:Conn_01x02 J?
+L Connector_Generic:Conn_01x02 J23
 U 1 1 5C071CEA
 P 7050 3600
-AR Path="/5BFF1764/5C071CEA" Ref="J?"  Part="1"
+AR Path="/5BFF1764/5C071CEA" Ref="J23"  Part="1"
 AR Path="/5C064586/5C071CEA" Ref="J?"  Part="1"
-F 0 "J?" H 7130 3592 50  0000 L CNN
+F 0 "J23" H 7130 3592 50  0000 L CNN
 F 1 "Mist" H 7130 3501 50  0000 L CNN
 F 2 "Connector_JST:JST_XH_S02B-XH-A-1_1x02_P2.50mm_Horizontal" H 7050 3600 50  0001 C CNN
@@
 	7400 3700 7400 4000
 $Comp
-L power:GND #PWR?
+L power:GND #PWR0126
 U 1 1 5C071CF4
 P 7400 4000
-F 0 "#PWR?" H 7400 3750 50  0001 C CNN
+F 0 "#PWR0126" H 7400 3750 50  0001 C CNN
 F 1 "GND" H 7450 3800 50  0000 C CNN
 F 2 "" H 7400 4000 50  0001 C CNN
@@
 $EndComp
 $Comp
-L Connector_Generic:Conn_01x02 J?
+L Connector_Generic:Conn_01x02 J22
 U 1 1 5C074870
 P 5750 3500
-AR Path="/5BFF1764/5C074870" Ref="J?"  Part="1"
+AR Path="/5BFF1764/5C074870" Ref="J22"  Part="1"
 AR Path="/5C064586/5C074870" Ref="J?"  Part="1"
-F 0 "J?" H 5830 3492 50  0000 L CNN
+F 0 "J22" H 5830 3492 50  0000 L CNN
 F 1 "Mist" H 5830 3401 50  0000 L CNN
 F 2 "Connector_JST:JST_XH_S02B-XH-A-1_1x02_P2.50mm_Horizontal" H 5750 3500 50  0001 C CNN
@@
 	6100 3600 6100 3900
 $Comp
-L power:GND #PWR?
+L power:GND #PWR0139
 U 1 1 5C07487A
 P 6100 3900
-F 0 "#PWR?" H 6100 3650 50  0001 C CNN
+F 0 "#PWR0139" H 6100 3650 50  0001 C CNN
 F 1 "GND" H 6150 3700 50  0000 C CNN
 F 2 "" H 6100 3900 50  0001 C CNN
@@
 $EndComp
 $Comp
-L Connector_Generic:Conn_01x02 J?
+L Connector_Generic:Conn_01x02 J10
 U 1 1 5C076A4A
 P 5750 2700
-AR Path="/5BFF1764/5C076A4A" Ref="J?"  Part="1"
+AR Path="/5BFF1764/5C076A4A" Ref="J10"  Part="1"
 AR Path="/5C064586/5C076A4A" Ref="J?"  Part="1"
-F 0 "J?" H 5830 2692 50  0000 L CNN
+F 0 "J10" H 5830 2692 50  0000 L CNN
 F 1 "Mist" H 5830 2601 50  0000 L CNN
 F 2 "Connector_JST:JST_XH_S02B-XH-A-1_1x02_P2.50mm_Horizontal" H 5750 2700 50  0001 C CNN
@@
 	6100 2800 6100 3100
 $Comp
-L power:GND #PWR?
+L power:GND #PWR0140
 U 1 1 5C076A54
 P 6100 3100
-F 0 "#PWR?" H 6100 2850 50  0001 C CNN
+F 0 "#PWR0140" H 6100 2850 50  0001 C CNN
 F 1 "GND" H 6150 2900 50  0000 C CNN
 F 2 "" H 6100 3100 50  0001 C CNN
