File: PWM.sch (KiCad schematic (older format))
At the start: 7 parts

Commit message: update,
Parts:
- removed D?: SD_1N4001_M1, symbol taobao-sd:SD_1N4001_M1
- added D2: SD_SS510, Diode_SMD:D_1206_3216Metric_Pad1.42x1.75mm_HandSolder, symbol taobao-sd:SD_SS510
- J20: renamed from J?; value Conn_01x02 -> PWM_TO_MOTOR; footprint (none) -> Connector_PinHeader_2.54mm:PinHeader_1x02_P2.54mm_Vertical
- gave numbers to parts that had none: 5
Connections:
- net +12V: now also D2.1 (K)
- net at J20.2 (Pin_2), Q1.2 (D): now also D2.2 (A)
Changed lines of the file:
@@
 $EndDescr
 $Comp
-L Transistor_FET:IRF540N Q?
+L Transistor_FET:IRF540N Q1
 U 1 1 5C066F82
 P 5900 3350
-F 0 "Q?" H 6105 3396 50  0000 L CNN
+F 0 "Q1" H 6105 3396 50  0000 L CNN
 F 1 "IRF540N" H 6105 3305 50  0000 L CNN
 F 2 "Package_TO_SOT_SMD:TO-263-2" H 6150 3275 50  0001 L CIN
@@
 $EndBitmap
 $Comp
-L taobao-r:R103,0805 R?
+L taobao-r:R103,0805 R5
 U 1 1 5C0675E7
 P 4900 3700
-F 0 "R?" H 4959 3746 50  0000 L CNN
+F 0 "R5" H 4959 3746 50  0000 L CNN
 F 1 "R103,0805" H 4959 3655 50  0000 L CNN
 F 2 "Resistor_SMD:R_0805_2012Metric_Pad1.15x1.40mm_HandSolder" H 4900 3700 50  0001 C CNN
@@
 $EndComp
 $Comp
-L power:GND #PWR?
+L power:GND #PWR0132
 U 1 1 5C067664
 P 5850 4150
-F 0 "#PWR?" H 5850 3900 50  0001 C CNN
+F 0 "#PWR0132" H 5850 3900 50  0001 C CNN
 F 1 "GND" H 5855 3977 50  0000 C CNN
 F 2 "" H 5850 4150 50  0001 C CNN
@@
 	3050 3150 3850 3150
 $Comp
-L Connector_Generic:Conn_01x02 J?
+L Connector_Generic:Conn_01x02 J20
 U 1 1 5C067E14
 P 6600 2650
-F 0 "J?" H 6680 2642 50  0000 L CNN
-F 1 "Conn_01x02" H 6680 2551 50  0000 L CNN
-F 2 "" H 6600 2650 50  0001 C CNN
+F 0 "J20" H 6680 2642 50  0000 L CNN
+F 1 "PWM_TO_MOTOR" H 6680 2551 50  0000 L CNN
+F 2 "Connector_PinHeader_2.54mm:PinHeader_1x02_P2.54mm_Vertical" H 6600 2650 50  0001 C CNN
 F 3 "~" H 6600 2650 50  0001 C CNN
 	1    6600 2650
@@
 $EndComp
 $Comp
-L power:+12V #PWR?
+L power:+12V #PWR0133
 U 1 1 5C067FCF
 P 6000 2350
-F 0 "#PWR?" H 6000 2200 50  0001 C CNN
+F 0 "#PWR0133" H 6000 2200 50  0001 C CNN
 F 1 "+12V" H 6015 2523 50  0000 C CNN
 F 2 "" H 6000 2350 50  0001 C CNN
@@
 	6000 2850 6000 2800
 $Comp
-L taobao-sd:SD_1N4001_M1 D?
-U 1 1 5C068BCE
-P 6000 2700
-F 0 "D?" V 5954 2633 50  0000 R CNN
-F 1 "SD_1N4001_M1" V 6045 2633 50  0000 R CNN
-F 2 "" V 6000 2700 50  0001 C CNN
-F 3 "~" V 6000 2700 50  0001 C CNN
-	1    6000 2700
-	0    1    1    0
-$EndComp
-$Comp
-L Isolator:4N35 U?
+L Isolator:4N35 U5
 U 1 1 5C06902C
 P 4500 3250
-F 0 "U?" H 4500 3575 50  0000 C CNN
+F 0 "U5" H 4500 3575 50  0000 C CNN
 F 1 "4N35" H 4500 3484 50  0000 C CNN
 F 2 "Package_DIP:DIP-6_W7.62mm" H 4300 3050 50  0001 L CIN
@@
 $EndComp
 $Comp
-L taobao-r:R330,0805 R?
+L taobao-r:R330,0805 R3
 U 1 1 5C06942B
 P 3950 3150
-F 0 "R?" V 3754 3150 50  0000 C CNN
+F 0 "R3" V 3754 3150 50  0000 C CNN
 F 1 "R330,0805" V 3845 3150 50  0000 C CNN
 F 2 "Resistor_SMD:R_0805_2012Metric_Pad1.15x1.40mm_HandSolder" H 3950 3150 50  0001 C CNN
@@
 	4900 3350 4900 3600
 $Comp
-L power:+12V #PWR?
+L power:+12V #PWR0134
 U 1 1 5C06AD0F
 P 4900 2250
-F 0 "#PWR?" H 4900 2100 50  0001 C CNN
+F 0 "#PWR0134" H 4900 2100 50  0001 C CNN
 F 1 "+12V" H 4915 2423 50  0000 C CNN
 F 2 "" H 4900 2250 50  0001 C CNN
@@
 	4900 2250 4900 2650
 $Comp
-L power:GND #PWR?
+L power:GND #PWR0135
 U 1 1 5C06B354
 P 4100 4100
-F 0 "#PWR?" H 4100 3850 50  0001 C CNN
+F 0 "#PWR0135" H 4100 3850 50  0001 C CNN
 F 1 "GND" H 4105 3927 50  0000 C CNN
 F 2 "" H 4100 4100 50  0001 C CNN
@@
 Connection ~ 4900 3350
 $Comp
-L taobao-r:R102,0805 R?
+L taobao-r:R102,0805 R4
 U 1 1 5C06C6B5
 P 4900 2750
-F 0 "R?" H 4959 2796 50  0000 L CNN
+F 0 "R4" H 4959 2796 50  0000 L CNN
 F 1 "R102,0805" H 4959 2705 50  0000 L CNN
 F 2 "Resistor_SMD:R_0805_2012Metric_Pad1.15x1.40mm_HandSolder" H 4900 2750 50  0001 C CNN
@@
 	1    0    0    -1
 $EndComp
+$Comp
+L taobao-sd:SD_SS510 D2
+U 1 1 5C07034B
+P 6000 2700
+F 0 "D2" V 5954 2768 50  0000 L CNN
+F 1 "SD_SS510" V 6045 2768 50  0000 L CNN
+F 2 "Diode_SMD:D_1206_3216Metric_Pad1.42x1.75mm_HandSolder" V 6000 2700 50  0001 C CNN
+F 3 "~" V 6000 2700 50  0001 C CNN
+	1    6000 2700
+	0    1    1    0
+$EndComp
 $EndSCHEMATC
