File: 12V_power_supply.sch (KiCad schematic (older format))
At the start: 0 parts

Commit message: update,
Parts:
- added C4: CP220uf,50V, Capacitor_SMD:CP_Elec_10x10.5, symbol taobao-cp:CP220uf,50V
- added C5, C6, C7: C105,0805, Capacitor_SMD:C_0805_2012Metric_Pad1.15x1.40mm_HandSolder, symbol taobao-c:C105,0805
- added C8: CP330uf,25V, Capacitor_SMD:CP_Elec_8x10.5, symbol taobao-cp:CP330uf,25V
- added D3: SD_SS510, Diode_SMD:D_1206_3216Metric_Pad1.42x1.75mm_HandSolder, symbol taobao-sd:SD_SS510
- added D4: SD_1N5817_SS12, Diode_SMD:D_1206_3216Metric_Pad1.42x1.75mm_HandSolder, symbol taobao-sd:SD_1N5817_SS12
- added J9: Barrel_Jack_Switch, Connector_BarrelJack:BarrelJack_Horizontal, symbol Connector:Barrel_Jack_Switch
- added L1: L_47UH,5A,1040, Inductor_SMD:L_Wuerth_HCI-1040, symbol taobao-l:L_47UH,5A,1040
- added R6: R103,0805, Resistor_SMD:R_0805_2012Metric_Pad1.15x1.40mm_HandSolder, symbol taobao-r:R103,0805
- added R7: R333,0805, Resistor_SMD:R_0805_2012Metric_Pad1.15x1.40mm_HandSolder, symbol taobao-r:R333,0805
- added R8: R332,0805, Resistor_SMD:R_0805_2012Metric_Pad1.15x1.40mm_HandSolder, symbol taobao-r:R332,0805
- added U6: XL4015, Package_TO_SOT_SMD:TO-263-5_TabPin3, symbol taobao-components:XL4015
Connections:
- new net: C6.2, U6.4 (VC)
- new net: D3.1 (K), L1.1, U6.3 (SW)
- new net: R6.1, R7.2, R8.1
- new net: D4.1 (K), R6.2, U6.2 (FB)
- new net +12V: C7.1, C8.1, L1.2, R7.1
- new net +24V: C4.1, C5.1, C6.1, J9.1, U6.5 (VIN)
- new net GND: C4.2, C5.2, C7.2, C8.2, D3.2 (A), D4.2 (A), J9.2, R8.2, U6.1 (GND)

Commit message: update,
Parts:
- added J?: Conn_01x02, Connector_PinHeader_2.54mm:PinHeader_1x02_P2.54mm_Vertical, symbol Connector_Generic:Conn_01x02
Connections:
- net +24V: now also J?.1 (Pin_1)
- net GND: now also J?.2 (Pin_2)
Changed lines of the file:
@@
 $EndComp
 Wire Wire Line
-	2850 3900 2850 4150
+	2850 3900 2850 4100
 Wire Wire Line
 	2850 4150 2600 4150
@@
 $EndComp
 Wire Wire Line
-	2850 4350 2850 4600
+	2850 4350 2850 4400
 Wire Wire Line
 	2600 4350 2850 4350
@@
 	1    0    0    -1
 $EndComp
+$Comp
+L Connector_Generic:Conn_01x02 J?
+U 1 1 5C070F19
+P 3300 4200
+F 0 "J?" H 3400 4200 50  0000 L CNN
+F 1 "Conn_01x02" H 3400 4100 50  0000 L CNN
+F 2 "Connector_PinHeader_2.54mm:PinHeader_1x02_P2.54mm_Vertical" H 3300 4200 50  0001 C CNN
+F 3 "~" H 3300 4200 50  0001 C CNN
+	1    3300 4200
+	1    0    0    -1
+$EndComp
+Wire Wire Line
+	2850 4100 3000 4100
+Wire Wire Line
+	3000 4100 3000 4200
+Wire Wire Line
+	3000 4200 3100 4200
+Connection ~ 2850 4100
+Wire Wire Line
+	2850 4100 2850 4150
+Wire Wire Line
+	2850 4400 3000 4400
+Wire Wire Line
+	3000 4400 3000 4300
+Wire Wire Line
+	3000 4300 3100 4300
+Connection ~ 2850 4400
+Wire Wire Line
+	2850 4400 2850 4600
 $EndSCHEMATC
