File: tryouts/test.kicad_pcb (KiCad board)
At the start: 2 copper layers, 100 x 70 mm, 22 parts, among them J1 Conn_01x02, J20 PWM_TO_MOTOR, J9 Barrel_Jack_Switch, Q1 IRF540N, U5 4N35, U6 XL4015

Commit message: update,
Parts:
- added C1: CP47uf,35V, w_smd_cap:c_elec_5x5.3, F.Cu at (60.1, 46.2)
- added C2: CP47uf,35V, w_smd_cap:c_elec_5x5.3, F.Cu at (82.6, 46.3)
- added D1: LED_GREEN, LED_SMD:LED_0805_2012Metric_Pad1.15x1.40mm_HandSolder, B.Cu at (14.4, 41.0)
- added J1: Conn_01x02, Connector_PinHeader_2.54mm:PinHeader_1x02_P2.54mm_Vertical, F.Cu at (9.00, 48.5)
- added J2: Conn_01x04, Connector_PinHeader_2.54mm:PinHeader_1x04_P2.54mm_Vertical, F.Cu at (14.5, 55.5)
- added J3: Conn_02x03_Odd_Even, Connector_PinHeader_2.54mm:PinHeader_2x03_P2.54mm_Vertical, F.Cu at (67.4, 47.4)
- added J4: Conn_02x03_Odd_Even, Connector_PinHeader_2.54mm:PinHeader_2x03_P2.54mm_Vertical, F.Cu at (89.7, 47.5)
- added J6: Conn_01x04, Connector_JST:JST_XH_S04B-XH-A-1_1x04_P2.50mm_Horizontal, F.Cu at (61.4, 60.2)
- added J7: Conn_01x04, Connector_JST:JST_XH_S04B-XH-A-1_1x04_P2.50mm_Horizontal, F.Cu at (84.6, 61.2)
- added R1: R103,0805, Resistor_SMD:R_0805_2012Metric_Pad1.15x1.40mm_HandSolder, B.Cu at (15.9, 46.5)
- added R2: R473,0805, Resistor_SMD:R_0805_2012Metric_Pad1.15x1.40mm_HandSolder, B.Cu at (12.9, 46.5)
- added R3: R102,0805, Resistor_SMD:R_0805_2012Metric_Pad1.15x1.40mm_HandSolder, B.Cu at (11.3, 34.9)
- added U1: arduino_nano_v3, footprint-lib:Arduino_Nano, F.Cu at (21.5, 27.0)
- added U2: 4N35, Package_DIP:DIP-6_W7.62mm, F.Cu at (8.00, 33.5)
- added U3: A4988_MODULE, Module:Pololu_Breakout-16_15.2x20.3mm, F.Cu at (74.1, 39.6)
- added U4: A4988_MODULE, Module:Pololu_Breakout-16_15.2x20.3mm, F.Cu at (97.2, 40.0)
- moved J9 25.3 mm to (59.0, 3.50)
- moved D2 1.41 mm to (42.9, 11.4)
- moved J1 1.41 mm to (4.31, 11.4)
- moved J20 1.41 mm to (45.8, 9.98)
- moved Q1 1.41 mm to (30.5, 12.3)
- moved R3 1.41 mm to (8.80, 4.96)
- moved R4 1.41 mm to (26.7, 5.13)
- moved R5 1.41 mm to (16.7, 14.5)
- moved U5 1.41 mm to (12.7, 5.18)
Routing:
- net +5V: track 0.00 -> 122.7 mm
- net GND: track 139.4 -> 226.7 mm
- net +VMot: track 0.00 -> 46.9 mm
- net Step_Enable: track 0.00 -> 24.1 mm
- net Net-(D1-Pad1): track 0.00 -> 17.1 mm, vias 0 -> 2
- net Net-(J1-Pad2): track 0.00 -> 16.3 mm
- net +12V: track 63.5 -> 73.4 mm
- net Net-(J7-Pad4): track 0.00 -> 8.54 mm
- net Net-(J7-Pad1): track 0.00 -> 8.53 mm
- net Net-(J7-Pad3): track 0.00 -> 8.53 mm
- net Net-(J7-Pad2): track 0.00 -> 8.51 mm
- net Net-(J6-Pad4): track 0.00 -> 7.92 mm
- net Net-(J6-Pad3): track 0.00 -> 7.90 mm
- net Net-(J6-Pad2): track 0.00 -> 7.89 mm
- net Net-(J6-Pad1): track 0.00 -> 7.87 mm
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