File: tryouts/POWER_SUPPLY/POWER_SUPPLY.sch (KiCad schematic (older format))
At the start: 18 parts

Commit message: update,
Parts:
- gave numbers to parts that had none: 18
Changed lines of the file:
@@
 EESchema Schematic File Version 4
+LIBS:POWER_SUPPLY-cache
 EELAYER 26 0
 EELAYER END
@@
 AR Path="/5BFF1764/5BFF4033" Ref="H?"  Part="1"
 AR Path="/5C064586/5BFF4033" Ref="H?"  Part="1"
-F 0 "H?" V 5900 7151 50  0000 L CNN
+AR Path="/5BFF4033" Ref="H1"  Part="1"
+F 0 "H1" V 5900 7151 50  0000 L CNN
 F 1 "MountingHole_Pad" V 5900 7060 50  0000 L CNN
 F 2 "MountingHole:MountingHole_2.7mm_M2.5_Pad" H 5800 7100 50  0001 C CNN
@@
 AR Path="/5BFF1764/5BFF40E1" Ref="H?"  Part="1"
 AR Path="/5C064586/5BFF40E1" Ref="H?"  Part="1"
-F 0 "H?" V 6200 7151 50  0000 L CNN
+AR Path="/5BFF40E1" Ref="H2"  Part="1"
+F 0 "H2" V 6200 7151 50  0000 L CNN
 F 1 "MountingHole_Pad" V 6200 7060 50  0000 L CNN
 F 2 "MountingHole:MountingHole_2.7mm_M2.5_Pad" H 6100 7100 50  0001 C CNN
@@
 AR Path="/5BFF1764/5BFF40FF" Ref="H?"  Part="1"
 AR Path="/5C064586/5BFF40FF" Ref="H?"  Part="1"
-F 0 "H?" V 6500 7151 50  0000 L CNN
+AR Path="/5BFF40FF" Ref="H3"  Part="1"
+F 0 "H3" V 6500 7151 50  0000 L CNN
 F 1 "MountingHole_Pad" V 6500 7060 50  0000 L CNN
 F 2 "MountingHole:MountingHole_2.7mm_M2.5_Pad" H 6400 7100 50  0001 C CNN
@@
 AR Path="/5BFF1764/5BFF4125" Ref="H?"  Part="1"
 AR Path="/5C064586/5BFF4125" Ref="H?"  Part="1"
-F 0 "H?" V 6750 7151 50  0000 L CNN
+AR Path="/5BFF4125" Ref="H4"  Part="1"
+F 0 "H4" V 6750 7151 50  0000 L CNN
 F 1 "MountingHole_Pad" V 6750 7060 50  0000 L CNN
 F 2 "MountingHole:MountingHole_2.7mm_M2.5_Pad" H 6650 7100 50  0001 C CNN
@@
 AR Path="/5BFF1764/5BFF421C" Ref="#PWR?"  Part="1"
 AR Path="/5C064586/5BFF421C" Ref="#PWR?"  Part="1"
-F 0 "#PWR?" H 6250 7150 50  0001 C CNN
+AR Path="/5BFF421C" Ref="#PWR0101"  Part="1"
+F 0 "#PWR0101" H 6250 7150 50  0001 C CNN
 F 1 "GND" H 6255 7227 50  0000 C CNN
 F 2 "" H 6250 7400 50  0001 C CNN
@@
 AR Path="/5BFF1764/5BFF8AAE" Ref="J?"  Part="1"
 AR Path="/5C064586/5BFF8AAE" Ref="J?"  Part="1"
-F 0 "J?" H 3020 4467 50  0000 C CNN
+AR Path="/5BFF8AAE" Ref="J11"  Part="1"
+F 0 "J11" H 3020 4467 50  0000 C CNN
 F 1 "MOTOR" H 3020 4376 50  0000 C CNN
 F 2 "Connector_JST:JST_XH_S05B-XH-A-1_1x05_P2.50mm_Horizontal" H 3100 4050 50  0001 C CNN
@@
 AR Path="/5BFF1764/5BFFB401" Ref="#PWR?"  Part="1"
 AR Path="/5C064586/5BFFB401" Ref="#PWR?"  Part="1"
-F 0 "#PWR?" H 4250 4000 50  0001 C CNN
+AR Path="/5BFFB401" Ref="#PWR0102"  Part="1"
+F 0 "#PWR0102" H 4250 4000 50  0001 C CNN
 F 1 "+5V" H 4265 4323 50  0000 C CNN
 F 2 "" H 4250 4150 50  0000 C CNN
@@
 AR Path="/5BFF1764/5BFFBFD9" Ref="#PWR?"  Part="1"
 AR Path="/5C064586/5BFFBFD9" Ref="#PWR?"  Part="1"
-F 0 "#PWR?" H 4150 3400 50  0001 C CNN
+AR Path="/5BFFBFD9" Ref="#PWR0103"  Part="1"
+F 0 "#PWR0103" H 4150 3400 50  0001 C CNN
 F 1 "GND" H 4155 3477 50  0000 C CNN
 F 2 "" H 4150 3650 50  0001 C CNN
@@
 AR Path="/5BFF1764/5C030BBA" Ref="J?"  Part="1"
 AR Path="/5C064586/5C030BBA" Ref="J?"  Part="1"
-F 0 "J?" H 9750 850 50  0000 C CNN
+AR Path="/5C030BBA" Ref="J1"  Part="1"
+F 0 "J1" H 9750 850 50  0000 C CNN
 F 1 "X_LIMIT1" H 9850 750 50  0000 C CNN
 F 2 "Connector_JST:JST_XH_S02B-XH-A-1_1x02_P2.50mm_Horizontal" H 9600 850 50  0001 C CNN
@@
 AR Path="/5BFF1764/5C0318FB" Ref="J?"  Part="1"
 AR Path="/5C064586/5C0318FB" Ref="J?"  Part="1"
-F 0 "J?" H 9680 1192 50  0000 L CNN
+AR Path="/5C0318FB" Ref="J2"  Part="1"
+F 0 "J2" H 9680 1192 50  0000 L CNN
 F 1 "Y_LIMIT1" H 9680 1101 50  0000 L CNN
 F 2 "Connector_JST:JST_XH_S02B-XH-A-1_1x02_P2.50mm_Horizontal" H 9600 1200 50  0001 C CNN
@@
 AR Path="/5BFF1764/5C031931" Ref="J?"  Part="1"
 AR Path="/5C064586/5C031931" Ref="J?"  Part="1"
-F 0 "J?" H 9680 1492 50  0000 L CNN
+AR Path="/5C031931" Ref="J3"  Part="1"
+F 0 "J3" H 9680 1492 50  0000 L CNN
 F 1 "Z_LIMIT1" H 9680 1401 50  0000 L CNN
 F 2 "Connector_JST:JST_XH_S02B-XH-A-1_1x02_P2.50mm_Horizontal" H 9600 1500 50  0001 C CNN
@@
 AR Path="/5BFF1764/5C03426F" Ref="J?"  Part="1"
 AR Path="/5C064586/5C03426F" Ref="J?"  Part="1"
-F 0 "J?" H 9680 4192 50  0000 L CNN
+AR Path="/5C03426F" Ref="J12"  Part="1"
+F 0 "J12" H 9680 4192 50  0000 L CNN
 F 1 "PROBE" H 9680 4101 50  0000 L CNN
 F 2 "Connector_JST:JST_XH_S02B-XH-A-1_1x02_P2.50mm_Horizontal" H 9600 4200 50  0001 C CNN
@@
 AR Path="/5BFF1764/5C0359F8" Ref="J?"  Part="1"
 AR Path="/5C064586/5C0359F8" Ref="J?"  Part="1"
-F 0 "J?" H 9680 4492 50  0000 L CNN
+AR Path="/5C0359F8" Ref="J13"  Part="1"
+F 0 "J13" H 9680 4492 50  0000 L CNN
 F 1 "START" H 9680 4401 50  0000 L CNN
 F 2 "Connector_JST:JST_XH_S02B-XH-A-1_1x02_P2.50mm_Horizontal" H 9600 4500 50  0001 C CNN
@@
 AR Path="/5BFF1764/5C03E431" Ref="J?"  Part="1"
 AR Path="/5C064586/5C03E431" Ref="J?"  Part="1"
-F 0 "J?" H 9680 4792 50  0000 L CNN
+AR Path="/5C03E431" Ref="J14"  Part="1"
+F 0 "J14" H 9680 4792 50  0000 L CNN
 F 1 "HOLD" H 9680 4701 50  0000 L CNN
 F 2 "Connector_JST:JST_XH_S02B-XH-A-1_1x02_P2.50mm_Horizontal" H 9600 4800 50  0001 C CNN
@@
 AR Path="/5BFF1764/5C03F42E" Ref="#PWR?"  Part="1"
 AR Path="/5C064586/5C03F42E" Ref="#PWR?"  Part="1"
-F 0 "#PWR?" H 9950 4900 50  0001 C CNN
+AR Path="/5C03F42E" Ref="#PWR0104"  Part="1"
+F 0 "#PWR0104" H 9950 4900 50  0001 C CNN
 F 1 "GND" H 9955 4977 50  0000 C CNN
 F 2 "" H 9950 5150 50  0001 C CNN
@@
 AR Path="/5BFF1764/5C0541C9" Ref="J?"  Part="1"
 AR Path="/5C064586/5C0541C9" Ref="J?"  Part="1"
-F 0 "J?" H 9700 2350 50  0000 C CNN
+AR Path="/5C0541C9" Ref="J4"  Part="1"
+F 0 "J4" H 9700 2350 50  0000 C CNN
 F 1 "X_LIMIT2" H 9800 2250 50  0000 C CNN
 F 2 "Connector_JST:JST_XH_S02B-XH-A-1_1x02_P2.50mm_Horizontal" H 9550 2350 50  0001 C CNN
@@
 AR Path="/5BFF1764/5C0541D2" Ref="J?"  Part="1"
 AR Path="/5C064586/5C0541D2" Ref="J?"  Part="1"
-F 0 "J?" H 9630 2692 50  0000 L CNN
+AR Path="/5C0541D2" Ref="J6"  Part="1"
+F 0 "J6" H 9630 2692 50  0000 L CNN
 F 1 "Y_LIMIT2" H 9630 2601 50  0000 L CNN
 F 2 "Connector_JST:JST_XH_S02B-XH-A-1_1x02_P2.50mm_Horizontal" H 9550 2700 50  0001 C CNN
@@
 AR Path="/5BFF1764/5C0541D8" Ref="J?"  Part="1"
 AR Path="/5C064586/5C0541D8" Ref="J?"  Part="1"
-F 0 "J?" H 9630 2992 50  0000 L CNN
+AR Path="/5C0541D8" Ref="J8"  Part="1"
+F 0 "J8" H 9630 2992 50  0000 L CNN
 F 1 "Z_LIMIT2" H 9630 2901 50  0000 L CNN
 F 2 "Connector_JST:JST_XH_S02B-XH-A-1_1x02_P2.50mm_Horizontal" H 9550 3000 50  0001 C CNN
@@
 AR Path="/5BFF1764/5C055B77" Ref="#PWR?"  Part="1"
 AR Path="/5C064586/5C055B77" Ref="#PWR?"  Part="1"
-F 0 "#PWR?" H 9950 1600 50  0001 C CNN
+AR Path="/5C055B77" Ref="#PWR0105"  Part="1"
+F 0 "#PWR0105" H 9950 1600 50  0001 C CNN
 F 1 "GND" H 9955 1677 50  0000 C CNN
 F 2 "" H 9950 1850 50  0001 C CNN
@@
 AR Path="/5BFF1764/5C0573EE" Ref="#PWR?"  Part="1"
 AR Path="/5C064586/5C0573EE" Ref="#PWR?"  Part="1"
-F 0 "#PWR?" H 9900 3100 50  0001 C CNN
+AR Path="/5C0573EE" Ref="#PWR0106"  Part="1"
+F 0 "#PWR0106" H 9900 3100 50  0001 C CNN
 F 1 "GND" H 9905 3177 50  0000 C CNN
 F 2 "" H 9900 3350 50  0001 C CNN
@@
 AR Path="/5BFF1764/5C06FF5E" Ref="J?"  Part="1"
 AR Path="/5C064586/5C06FF5E" Ref="J?"  Part="1"
-F 0 "J?" H 7130 2742 50  0000 L CNN
+AR Path="/5C06FF5E" Ref="J7"  Part="1"
+F 0 "J7" H 7130 2742 50  0000 L CNN
 F 1 "Mist" H 7130 2651 50  0000 L CNN
 F 2 "Connector_JST:JST_XH_S02B-XH-A-1_1x02_P2.50mm_Horizontal" H 7050 2750 50  0001 C CNN
@@
 	7400 2850 7400 3150
 $Comp
-L power:GND #PWR?
+L power:GND #PWR0107
 U 1 1 5C0719A4
 P 7400 3150
-F 0 "#PWR?" H 7400 2900 50  0001 C CNN
+F 0 "#PWR0107" H 7400 2900 50  0001 C CNN
 F 1 "GND" H 7450 2950 50  0000 C CNN
 F 2 "" H 7400 3150 50  0001 C CNN
@@
 AR Path="/5BFF1764/5C071CEA" Ref="J?"  Part="1"
 AR Path="/5C064586/5C071CEA" Ref="J?"  Part="1"
-F 0 "J?" H 7130 3592 50  0000 L CNN
+AR Path="/5C071CEA" Ref="J10"  Part="1"
+F 0 "J10" H 7130 3592 50  0000 L CNN
 F 1 "Mist" H 7130 3501 50  0000 L CNN
 F 2 "Connector_JST:JST_XH_S02B-XH-A-1_1x02_P2.50mm_Horizontal" H 7050 3600 50  0001 C CNN
@@
 	7400 3700 7400 4000
 $Comp
-L power:GND #PWR?
+L power:GND #PWR0108
 U 1 1 5C071CF4
 P 7400 4000
-F 0 "#PWR?" H 7400 3750 50  0001 C CNN
+F 0 "#PWR0108" H 7400 3750 50  0001 C CNN
 F 1 "GND" H 7450 3800 50  0000 C CNN
 F 2 "" H 7400 4000 50  0001 C CNN
@@
 AR Path="/5BFF1764/5C074870" Ref="J?"  Part="1"
 AR Path="/5C064586/5C074870" Ref="J?"  Part="1"
-F 0 "J?" H 5830 3492 50  0000 L CNN
+AR Path="/5C074870" Ref="J9"  Part="1"
+F 0 "J9" H 5830 3492 50  0000 L CNN
 F 1 "Mist" H 5830 3401 50  0000 L CNN
 F 2 "Connector_JST:JST_XH_S02B-XH-A-1_1x02_P2.50mm_Horizontal" H 5750 3500 50  0001 C CNN
@@
 	6100 3600 6100 3900
 $Comp
-L power:GND #PWR?
+L power:GND #PWR0109
 U 1 1 5C07487A
 P 6100 3900
-F 0 "#PWR?" H 6100 3650 50  0001 C CNN
+F 0 "#PWR0109" H 6100 3650 50  0001 C CNN
 F 1 "GND" H 6150 3700 50  0000 C CNN
 F 2 "" H 6100 3900 50  0001 C CNN
@@
 AR Path="/5BFF1764/5C076A4A" Ref="J?"  Part="1"
 AR Path="/5C064586/5C076A4A" Ref="J?"  Part="1"
-F 0 "J?" H 5830 2692 50  0000 L CNN
+AR Path="/5C076A4A" Ref="J5"  Part="1"
+F 0 "J5" H 5830 2692 50  0000 L CNN
 F 1 "Mist" H 5830 2601 50  0000 L CNN
 F 2 "Connector_JST:JST_XH_S02B-XH-A-1_1x02_P2.50mm_Horizontal" H 5750 2700 50  0001 C CNN
@@
 	6100 2800 6100 3100
 $Comp
-L power:GND #PWR?
+L power:GND #PWR0110
 U 1 1 5C076A54
 P 6100 3100
-F 0 "#PWR?" H 6100 2850 50  0001 C CNN
+F 0 "#PWR0110" H 6100 2850 50  0001 C CNN
 F 1 "GND" H 6150 2900 50  0000 C CNN
 F 2 "" H 6100 3100 50  0001 C CNN
